Commit message: Add additional links and joints to ak45.urdf.xacro

File: src/marsworks_ak45/urdf/ak45.urdf.xacro (robot description, xacro)
@@ -1,13 +1,32 @@
 <?xml version="1.0"?>
 <robot xmlns:xacro="http://www.ros.org/wiki/xacro" name="ak45">
+  <!-- Links -->
   <link name="base_link"/>
-  <link name="output_link"/>
-  <joint name="ak45_joint" type="revolute">
+  <link name="link_1"/>
+  <link name="link_2"/>
+  <link name="link_3"/>
+  <!-- Joints -->
+  <joint name="joint_1" type="revolute">
     <parent link="base_link"/>
-    <child link="output_link"/>
+    <child link="link_1"/>
     <origin xyz="0 0 0" rpy="0 0 0"/>
     <axis xyz="0 0 1"/>
     <limit lower="-3.14159" upper="3.14159" effort="24.0" velocity="5.44"/>
   </joint>
+  <joint name="joint_2" type="revolute">
+    <parent link="link_1"/>
+    <child link="link_2"/>
+    <origin xyz="0 0 0.1" rpy="0 0 0"/>
+    <axis xyz="0 0 1"/>
+    <limit lower="-3.14159" upper="3.14159" effort="24.0" velocity="5.44"/>
+  </joint>
+  <joint name="joint_3" type="revolute">
+    <parent link="link_2"/>
+    <child link="link_3"/>
+    <origin xyz="0 0 0.1" rpy="0 0 0"/>
+    <axis xyz="0 0 1"/>
+    <limit lower="-3.14159" upper="3.14159" effort="24.0" velocity="5.44"/>
+  </joint>
+  <!-- ros2_control -->
   <ros2_control name="ak45_system" type="system">
     <hardware>
@@ -15,6 +34,6 @@
       <param name="can_interface">vcan0</param>
     </hardware>
-    <joint name="ak45_joint">
-      <param name="can_id">111</param>
+    <joint name="joint_1">
+      <param name="can_id">10</param>
       <param name="pole_pairs">14</param>
       <param name="gear_ratio">36</param>
@@ -24,5 +43,24 @@
       <state_interface name="velocity"/>
       <state_interface name="effort"/>
-      <state_interface name="temperature"/>
+    </joint>
+    <joint name="joint_2">
+      <param name="can_id">30</param>
+      <param name="pole_pairs">14</param>
+      <param name="gear_ratio">36</param>
+      <param name="kt">0.11</param>
+      <command_interface name="position"/>
+      <state_interface name="position"/>
+      <state_interface name="velocity"/>
+      <state_interface name="effort"/>
+    </joint>
+    <joint name="joint_3">
+      <param name="can_id">20</param>
+      <param name="pole_pairs">14</param>
+      <param name="gear_ratio">36</param>
+      <param name="kt">0.11</param>
+      <command_interface name="position"/>
+      <state_interface name="position"/>
+      <state_interface name="velocity"/>
+      <state_interface name="effort"/>
     </joint>
   </ros2_control>

Commit message: modified code

File: src/marsworks_ak45/urdf/ak45.urdf.xacro (robot description, xacro)
@@ -2,8 +2,32 @@
 <robot xmlns:xacro="http://www.ros.org/wiki/xacro" name="ak45">
   <link name="base_link"/>
-  <link name="output_link"/>
-  <joint name="ak45_joint" type="revolute">
+  <link name="motor_1_output"/>
+  <link name="motor_2_output"/>
+  <link name="motor_3_output"/>
+  <link name="motor_4_output"/>
+  <joint name="motor_1" type="revolute">
     <parent link="base_link"/>
-    <child link="output_link"/>
+    <child link="motor_1_output"/>
+    <origin xyz="0 0 0" rpy="0 0 0"/>
+    <axis xyz="0 0 1"/>
+    <limit lower="-3.14159" upper="3.14159" effort="24.0" velocity="5.44"/>
+  </joint>
+  <joint name="motor_2" type="revolute">
+    <parent link="base_link"/>
+    <child link="motor_2_output"/>
+    <origin xyz="0 0 0" rpy="0 0 0"/>
+    <axis xyz="0 0 1"/>
+    <limit lower="-3.14159" upper="3.14159" effort="24.0" velocity="5.44"/>
+  </joint>
+  <joint name="motor_3" type="revolute">
+    <parent link="base_link"/>
+    <child link="motor_3_output"/>
+    <origin xyz="0 0 0" rpy="0 0 0"/>
+    <axis xyz="0 0 1"/>
+    <limit lower="-3.14159" upper="3.14159" effort="24.0" velocity="5.44"/>
+  </joint>
+  <joint name="motor_4" type="revolute">
+    <parent link="base_link"/>
+    <child link="motor_4_output"/>
     <origin xyz="0 0 0" rpy="0 0 0"/>
     <axis xyz="0 0 1"/>
@@ -13,12 +37,49 @@
     <hardware>
       <plugin>cubemars_hardware/CubeMarsSystemHardware</plugin>
-      <param name="can_interface">vcan0</param>
+      <param name="can_interface">can0</param>
     </hardware>
-    <joint name="ak45_joint">
+    <joint name="motor_1">
       <param name="can_id">111</param>
-      <param name="pole_pairs">14</param>
-      <param name="gear_ratio">36</param>
-      <param name="kt">0.11</param>
+      <param name="pole_pairs">21</param>
+      <param name="gear_ratio">9</param>
+      <param name="kt">0.198</param>
       <command_interface name="position"/>
+      <command_interface name="velocity"/>
+      <state_interface name="position"/>
+      <state_interface name="velocity"/>
+      <state_interface name="effort"/>
+      <state_interface name="temperature"/>
+    </joint>
+    <joint name="motor_2">
+      <param name="can_id">112</param>
+      <param name="pole_pairs">21</param>
+      <param name="gear_ratio">9</param>
+      <param name="kt">0.198</param>
+      <command_interface name="position"/>
+      <command_interface name="velocity"/>
+      <state_interface name="position"/>
+      <state_interface name="velocity"/>
+      <state_interface name="effort"/>
+      <state_interface name="temperature"/>
+    </joint>
+    <joint name="motor_3">
+      <param name="can_id">113</param>
+      <param name="pole_pairs">21</param>
+      <param name="gear_ratio">9</param>
+      <param name="kt">0.198</param>
+      <command_interface name="position"/>
+      <command_interface name="velocity"/>
+      <state_interface name="position"/>
+      <state_interface name="velocity"/>
+      <state_interface name="effort"/>
+      <state_interface name="temperature"/>
+    </joint>
+    <joint name="motor_4">
+      <param name="can_id">114</param>
+      <param name="pole_pairs">21</param>
+      <param name="gear_ratio">9</param>
+      <param name="kt">0.198</param>
+      <command_interface name="position"/>
+      <command_interface name="velocity"/>
       <state_interface name="position"/>
       <state_interface name="velocity"/>
